File: connectors.kicad_sch (KiCad schematic)
At the start: 9 parts, among them J3 Battery Pack, J4 Rotor Servo 1, J5 Rotor Servo 2, J6 Main Rotor ESC, J7 Tail Rotor ESC, J8 UART, J9 I2C

Commit message: Assign footprints to symbols
Parts:
- J2: renamed from J3; footprint (none) -> Connector_PinHeader_2.54mm:PinHeader_1x02_P2.54mm_Vertical
- J3: renamed from J4; footprint (none) -> Connector_PinHeader_2.54mm:PinHeader_1x03_P2.54mm_Vertical
- J4: renamed from J5; footprint (none) -> Connector_PinHeader_2.54mm:PinHeader_1x03_P2.54mm_Vertical
- J5: renamed from J6; footprint (none) -> Connector_PinHeader_2.54mm:PinHeader_1x03_P2.54mm_Vertical
- J6: renamed from J7; footprint (none) -> Connector_PinHeader_2.54mm:PinHeader_1x03_P2.54mm_Vertical
- J7: renamed from J9; footprint (none) -> Connector_PinHeader_2.54mm:PinHeader_1x02_P2.54mm_Vertical
- J8: footprint (none) -> Connector_PinHeader_2.54mm:PinHeader_1x02_P2.54mm_Vertical
- renumbered R9 to R4, R10 to R5
Other:
- moved on the sheet: J2, J3, J4, J5, J6, J7, J8, R4, R5
