File: communication.kicad_sch (KiCad schematic)
At the start: 2 parts

Commit message: Connect sensors to the MCU
Parts:
- gave numbers to parts that had none: 2
Changed lines of the file:
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@@
 (kicad_sch (version 20211123) (generator eeschema)
   (paper "A4")
+  (title_block
+    (date "2022-12-16")
+    (rev "0.1.0")
+  )
   (junction (at 149.86 81.28) (diameter 0) (color 0 0 0 0)
   )
@@
   (symbol (lib_id "power:+3.3V") (at 149.86 80.01 0) (unit 1)
     (in_bom yes) (on_board yes) (fields_autoplaced)
-    (property "Reference" "#PWR?" (id 0) (at 149.86 83.82 0)
+    (property "Reference" "#PWR0149" (id 0) (at 149.86 83.82 0)
       (effects (font (size 1.27 1.27)) hide)
     )
@@
   (symbol (lib_id "power:GND") (at 149.86 115.57 0) (unit 1)
     (in_bom yes) (on_board yes) (fields_autoplaced)
-    (property "Reference" "#PWR?" (id 0) (at 149.86 121.92 0)
+    (property "Reference" "#PWR0148" (id 0) (at 149.86 121.92 0)
       (effects (font (size 1.27 1.27)) hide)
     )
@@
   (symbol (lib_id "Device:C") (at 167.64 97.79 0) (unit 1)
     (in_bom yes) (on_board yes) (fields_autoplaced)
-    (property "Reference" "C?" (id 0) (at 171.45 96.5199 0)
+    (property "Reference" "C19" (id 0) (at 171.45 96.5199 0)
       (effects (font (size 1.27 1.27)) (justify left))
     )
@@
   (symbol (lib_id "RF:NRF24L01_Breakout") (at 149.86 97.79 0) (unit 1)
     (in_bom yes) (on_board yes)
-    (property "Reference" "U?" (id 0) (at 140.97 85.09 0)
+    (property "Reference" "U6" (id 0) (at 140.97 85.09 0)
       (effects (font (size 1.27 1.27)) (justify left))
     )

Commit message: Improve the power section:
- add ADC circuit to measure battery level
- add 5V LDO regulator
Parts:
- renumbered C19 to C21, U6 to U8
Other:
- title: (none) -> Communication
Changed lines of the file:
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@@
   (paper "A4")
   (title_block
-    (date "2022-12-16")
+    (title "Communication")
+    (date "2022-12-17")
     (rev "0.1.0")
   )
@@
   (symbol (lib_id "power:+3.3V") (at 149.86 80.01 0) (unit 1)
     (in_bom yes) (on_board yes) (fields_autoplaced)
-    (property "Reference" "#PWR0149" (id 0) (at 149.86 83.82 0)
+    (property "Reference" "#PWR053" (id 0) (at 149.86 83.82 0)
       (effects (font (size 1.27 1.27)) hide)
     )
@@
   (symbol (lib_id "power:GND") (at 149.86 115.57 0) (unit 1)
     (in_bom yes) (on_board yes) (fields_autoplaced)
-    (property "Reference" "#PWR0148" (id 0) (at 149.86 121.92 0)
+    (property "Reference" "#PWR054" (id 0) (at 149.86 121.92 0)
       (effects (font (size 1.27 1.27)) hide)
     )
@@
   (symbol (lib_id "Device:C") (at 167.64 97.79 0) (unit 1)
     (in_bom yes) (on_board yes) (fields_autoplaced)
-    (property "Reference" "C19" (id 0) (at 171.45 96.5199 0)
+    (property "Reference" "C21" (id 0) (at 171.45 96.5199 0)
       (effects (font (size 1.27 1.27)) (justify left))
     )
@@
   (symbol (lib_id "RF:NRF24L01_Breakout") (at 149.86 97.79 0) (unit 1)
     (in_bom yes) (on_board yes)
-    (property "Reference" "U6" (id 0) (at 140.97 85.09 0)
+    (property "Reference" "U8" (id 0) (at 140.97 85.09 0)
       (effects (font (size 1.27 1.27)) (justify left))
     )

Commit message: Assign footprints to symbols
Parts:
- removed C21: 10μF, symbol Device:C
- added C16: 10μF, Capacitor_SMD:C_0603_1608Metric, symbol Device:C_Small
- renumbered U8 to U6
Connections:
- net +3.3V: now also C16.1
- net GND: now also C16.2
Changed lines of the file:
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@@
     (title "Communication")
     (date "2022-12-17")
-    (rev "0.1.0")
+    (rev "${REVISION}")
   )
-  (junction (at 149.86 81.28) (diameter 0) (color 0 0 0 0)
-  )
-  (junction (at 149.86 114.3) (diameter 0) (color 0 0 0 0)
-  )
-  (wire (pts (xy 167.64 101.6) (xy 167.64 114.3))
+  (wire (pts (xy 175.26 93.98) (xy 175.26 95.25))
     (stroke (width 0) (type default) (color 0 0 0 0))
   )
@@
     (stroke (width 0) (type default) (color 0 0 0 0))
   )
-  (wire (pts (xy 149.86 80.01) (xy 149.86 81.28))
+  (wire (pts (xy 149.86 80.01) (xy 149.86 82.55))
     (stroke (width 0) (type default) (color 0 0 0 0))
   )
-  (wire (pts (xy 149.86 113.03) (xy 149.86 114.3))
+  (wire (pts (xy 149.86 113.03) (xy 149.86 115.57))
     (stroke (width 0) (type default) (color 0 0 0 0))
   )
@@
     (stroke (width 0) (type default) (color 0 0 0 0))
   )
-  (wire (pts (xy 149.86 81.28) (xy 149.86 82.55))
-    (stroke (width 0) (type default) (color 0 0 0 0))
-  )
   (wire (pts (xy 137.16 90.17) (xy 135.89 90.17))
     (stroke (width 0) (type default) (color 0 0 0 0))
   )
-  (wire (pts (xy 167.64 114.3) (xy 149.86 114.3))
-    (stroke (width 0) (type default) (color 0 0 0 0))
-  )
-  (wire (pts (xy 149.86 114.3) (xy 149.86 115.57))
-    (stroke (width 0) (type default) (color 0 0 0 0))
-  )
-  (wire (pts (xy 149.86 81.28) (xy 167.64 81.28))
+  (wire (pts (xy 175.26 100.33) (xy 175.26 102.87))
     (stroke (width 0) (type default) (color 0 0 0 0))
   )
   (wire (pts (xy 137.16 97.79) (xy 135.89 97.79))
-    (stroke (width 0) (type default) (color 0 0 0 0))
-  )
-  (wire (pts (xy 167.64 81.28) (xy 167.64 93.98))
     (stroke (width 0) (type default) (color 0 0 0 0))
   )
@@
     (effects (font (size 1.27 1.27)) (justify right))
   )
+  (symbol (lib_id "Device:C_Small") (at 175.26 97.79 0) (unit 1)
+    (in_bom yes) (on_board yes)
+    (property "Reference" "C16" (id 0) (at 177.5968 96.6216 0)
+      (effects (font (size 1.27 1.27)) (justify left))
+    )
+    (property "Value" "10μF" (id 1) (at 177.5968 98.933 0)
+      (effects (font (size 1.27 1.27)) (justify left))
+    )
+    (property "Footprint" "Capacitor_SMD:C_0603_1608Metric" (id 2) (at 175.26 97.79 0)
+      (effects (font (size 1.27 1.27)) hide)
+    )
+    (property "Datasheet" "~" (id 3) (at 175.26 97.79 0)
+      (effects (font (size 1.27 1.27)) hide)
+    )
+    (property "LCSC" "C19666" (id 4) (at 175.26 97.79 0)
+      (effects (font (size 1.27 1.27)) hide)
+    )
+    (pin "1")
+    (pin "2")
+  )
   (symbol (lib_id "power:+3.3V") (at 149.86 80.01 0) (unit 1)
     (in_bom yes) (on_board yes) (fields_autoplaced)
-    (property "Reference" "#PWR054" (id 0) (at 149.86 83.82 0)
+    (property "Reference" "#PWR040" (id 0) (at 149.86 83.82 0)
       (effects (font (size 1.27 1.27)) hide)
     )
@@
     (pin "1")
   )
+  (symbol (lib_id "power:+3.3V") (at 175.26 93.98 0) (unit 1)
+    (in_bom yes) (on_board yes) (fields_autoplaced)
+    (property "Reference" "#PWR?" (id 0) (at 175.26 97.79 0)
+      (effects (font (size 1.27 1.27)) hide)
+    )
+    (property "Value" "+3.3V" (id 1) (at 175.26 88.9 0))
+    (property "Footprint" "" (id 2) (at 175.26 93.98 0)
+      (effects (font (size 1.27 1.27)) hide)
+    )
+    (property "Datasheet" "" (id 3) (at 175.26 93.98 0)
+      (effects (font (size 1.27 1.27)) hide)
+    )
+    (pin "1")
+  )
   (symbol (lib_id "power:GND") (at 149.86 115.57 0) (unit 1)
     (in_bom yes) (on_board yes) (fields_autoplaced)
-    (property "Reference" "#PWR055" (id 0) (at 149.86 121.92 0)
+    (property "Reference" "#PWR041" (id 0) (at 149.86 121.92 0)
       (effects (font (size 1.27 1.27)) hide)
     )
@@
     (pin "1")
   )
-  (symbol (lib_id "Device:C") (at 167.64 97.79 0) (unit 1)
-    (in_bom yes) (on_board yes) (fields_autoplaced)
-    (property "Reference" "C21" (id 0) (at 171.45 96.5199 0)
-      (effects (font (size 1.27 1.27)) (justify left))
-    )
-    (property "Value" "10μF" (id 1) (at 171.45 99.0599 0)
-      (effects (font (size 1.27 1.27)) (justify left))
-    )
-    (property "Footprint" "" (id 2) (at 168.6052 101.6 0)
+  (symbol (lib_id "power:GND") (at 175.26 102.87 0) (unit 1)
+    (in_bom yes) (on_board yes)
+    (property "Reference" "#PWR?" (id 0) (at 175.26 109.22 0)
       (effects (font (size 1.27 1.27)) hide)
     )
-    (property "Datasheet" "~" (id 3) (at 167.64 97.79 0)
+    (property "Value" "GND" (id 1) (at 175.387 107.2642 0))
+    (property "Footprint" "" (id 2) (at 175.26 102.87 0)
+      (effects (font (size 1.27 1.27)) hide)
+    )
+    (property "Datasheet" "" (id 3) (at 175.26 102.87 0)
       (effects (font (size 1.27 1.27)) hide)
     )
     (pin "1")
-    (pin "2")
   )
   (symbol (lib_id "RF:NRF24L01_Breakout") (at 149.86 97.79 0) (unit 1)
     (in_bom yes) (on_board yes)
-    (property "Reference" "U8" (id 0) (at 140.97 85.09 0)
+    (property "Reference" "U6" (id 0) (at 140.97 85.09 0)
       (effects (font (size 1.27 1.27)) (justify left))
     )

Commit message: Use single connector for I/O
Parts:
- renumbered C16 to C17
Changed lines of the file:
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@@
   (title_block
     (title "Communication")
-    (date "2022-12-17")
+    (date "2022-12-20")
     (rev "${REVISION}")
   )
@@
   (symbol (lib_id "Device:C_Small") (at 175.26 97.79 0) (unit 1)
     (in_bom yes) (on_board yes)
-    (property "Reference" "C16" (id 0) (at 177.5968 96.6216 0)
+    (property "Reference" "C17" (id 0) (at 177.5968 96.6216 0)
       (effects (font (size 1.27 1.27)) (justify left))
     )
@@
   (symbol (lib_id "power:+3.3V") (at 149.86 80.01 0) (unit 1)
     (in_bom yes) (on_board yes) (fields_autoplaced)
-    (property "Reference" "#PWR040" (id 0) (at 149.86 83.82 0)
+    (property "Reference" "#PWR036" (id 0) (at 149.86 83.82 0)
       (effects (font (size 1.27 1.27)) hide)
     )
@@
   (symbol (lib_id "power:+3.3V") (at 175.26 93.98 0) (unit 1)
     (in_bom yes) (on_board yes) (fields_autoplaced)
-    (property "Reference" "#PWR?" (id 0) (at 175.26 97.79 0)
+    (property "Reference" "#PWR037" (id 0) (at 175.26 97.79 0)
       (effects (font (size 1.27 1.27)) hide)
     )
@@
   (symbol (lib_id "power:GND") (at 149.86 115.57 0) (unit 1)
     (in_bom yes) (on_board yes) (fields_autoplaced)
-    (property "Reference" "#PWR041" (id 0) (at 149.86 121.92 0)
+    (property "Reference" "#PWR039" (id 0) (at 149.86 121.92 0)
       (effects (font (size 1.27 1.27)) hide)
     )
@@
   (symbol (lib_id "power:GND") (at 175.26 102.87 0) (unit 1)
     (in_bom yes) (on_board yes)
-    (property "Reference" "#PWR?" (id 0) (at 175.26 109.22 0)
+    (property "Reference" "#PWR038" (id 0) (at 175.26 109.22 0)
       (effects (font (size 1.27 1.27)) hide)
     )
@@
       (effects (font (size 1.27 1.27) italic) (justify left) hide)
     )
-    (property "Datasheet" "http://www.nordicsemi.com/eng/content/download/2730/34105/file/nRF24L01_Product_Specification_v2_0.pdf" (id 3) (at 149.86 100.33 0)
+    (property "Datasheet" "https://datasheet.ciiva.com/18385/83-15187-18385942.pdf" (id 3) (at 149.86 100.33 0)
       (effects (font (size 1.27 1.27)) hide)
     )

Commit message: Remove 5V LDO regulator
Parts:
- removed C17: 10μF, Capacitor_SMD:C_0603_1608Metric, symbol Device:C_Small
- added C15: 10μF, Capacitor_Tantalum_SMD:CP_EIA-3216-10_Kemet-I, symbol Device:C_Polarized_Small
- renumbered U6 to U5
Connections:
- net +3.3V: now also C15.1
- net GND: now also C15.2
Changed lines of the file:
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@@
     (effects (font (size 1.27 1.27)) (justify right))
-  )
-  (symbol (lib_id "Device:C_Small") (at 175.26 97.79 0) (unit 1)
-    (in_bom yes) (on_board yes)
-    (property "Reference" "C17" (id 0) (at 177.5968 96.6216 0)
-      (effects (font (size 1.27 1.27)) (justify left))
-    )
-    (property "Value" "10μF" (id 1) (at 177.5968 98.933 0)
-      (effects (font (size 1.27 1.27)) (justify left))
-    )
-    (property "Footprint" "Capacitor_SMD:C_0603_1608Metric" (id 2) (at 175.26 97.79 0)
-      (effects (font (size 1.27 1.27)) hide)
-    )
-    (property "Datasheet" "~" (id 3) (at 175.26 97.79 0)
-      (effects (font (size 1.27 1.27)) hide)
-    )
-    (property "LCSC" "C19666" (id 4) (at 175.26 97.79 0)
-      (effects (font (size 1.27 1.27)) hide)
-    )
-    (pin "1")
-    (pin "2")
   )
   (symbol (lib_id "power:+3.3V") (at 149.86 80.01 0) (unit 1)
     (in_bom yes) (on_board yes) (fields_autoplaced)
-    (property "Reference" "#PWR036" (id 0) (at 149.86 83.82 0)
+    (property "Reference" "#PWR035" (id 0) (at 149.86 83.82 0)
       (effects (font (size 1.27 1.27)) hide)
     )
@@
   (symbol (lib_id "power:+3.3V") (at 175.26 93.98 0) (unit 1)
     (in_bom yes) (on_board yes) (fields_autoplaced)
-    (property "Reference" "#PWR037" (id 0) (at 175.26 97.79 0)
+    (property "Reference" "#PWR036" (id 0) (at 175.26 97.79 0)
       (effects (font (size 1.27 1.27)) hide)
     )
@@
   (symbol (lib_id "power:GND") (at 149.86 115.57 0) (unit 1)
     (in_bom yes) (on_board yes) (fields_autoplaced)
-    (property "Reference" "#PWR039" (id 0) (at 149.86 121.92 0)
+    (property "Reference" "#PWR038" (id 0) (at 149.86 121.92 0)
       (effects (font (size 1.27 1.27)) hide)
     )
@@
     (pin "1")
   )
+  (symbol (lib_id "Device:C_Polarized_Small") (at 175.26 97.79 0) (unit 1)
+    (in_bom yes) (on_board yes) (fields_autoplaced)
+    (property "Reference" "C15" (id 0) (at 177.8 95.9738 0)
+      (effects (font (size 1.27 1.27)) (justify left))
+    )
+    (property "Value" "10μF" (id 1) (at 177.8 98.5138 0)
+      (effects (font (size 1.27 1.27)) (justify left))
+    )
+    (property "Footprint" "Capacitor_Tantalum_SMD:CP_EIA-3216-10_Kemet-I" (id 2) (at 175.26 97.79 0)
+      (effects (font (size 1.27 1.27)) hide)
+    )
+    (property "Datasheet" "~" (id 3) (at 175.26 97.79 0)
+      (effects (font (size 1.27 1.27)) hide)
+    )
+    (pin "1")
+    (pin "2")
+  )
   (symbol (lib_id "power:GND") (at 175.26 102.87 0) (unit 1)
     (in_bom yes) (on_board yes)
-    (property "Reference" "#PWR038" (id 0) (at 175.26 109.22 0)
+    (property "Reference" "#PWR037" (id 0) (at 175.26 109.22 0)
       (effects (font (size 1.27 1.27)) hide)
     )
@@
   (symbol (lib_id "RF:NRF24L01_Breakout") (at 149.86 97.79 0) (unit 1)
     (in_bom yes) (on_board yes)
-    (property "Reference" "U6" (id 0) (at 140.97 85.09 0)
+    (property "Reference" "U5" (id 0) (at 140.97 85.09 0)
       (effects (font (size 1.27 1.27)) (justify left))
     )

Commit message: Arrange footprints
Parts:
- renumbered C15 to C16
Other:
- company: (none) -> Authors: H. Fedarovich, I. Kajdan
Changed lines of the file:
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@@
   (title_block
     (title "Communication")
-    (date "2022-12-20")
+    (date "2022-12-23")
     (rev "${REVISION}")
+    (company "Authors: H. Fedarovich, I. Kajdan")
+    (comment 1 "Reviewer: A. Bondyra")
   )
   (wire (pts (xy 175.26 93.98) (xy 175.26 95.25))
@@
   (symbol (lib_id "power:+3.3V") (at 149.86 80.01 0) (unit 1)
     (in_bom yes) (on_board yes) (fields_autoplaced)
-    (property "Reference" "#PWR035" (id 0) (at 149.86 83.82 0)
+    (property "Reference" "#PWR036" (id 0) (at 149.86 83.82 0)
       (effects (font (size 1.27 1.27)) hide)
     )
@@
   (symbol (lib_id "power:+3.3V") (at 175.26 93.98 0) (unit 1)
     (in_bom yes) (on_board yes) (fields_autoplaced)
-    (property "Reference" "#PWR036" (id 0) (at 175.26 97.79 0)
+    (property "Reference" "#PWR037" (id 0) (at 175.26 97.79 0)
       (effects (font (size 1.27 1.27)) hide)
     )
@@
   (symbol (lib_id "power:GND") (at 149.86 115.57 0) (unit 1)
     (in_bom yes) (on_board yes) (fields_autoplaced)
-    (property "Reference" "#PWR038" (id 0) (at 149.86 121.92 0)
+    (property "Reference" "#PWR039" (id 0) (at 149.86 121.92 0)
       (effects (font (size 1.27 1.27)) hide)
     )
@@
   (symbol (lib_id "Device:C_Polarized_Small") (at 175.26 97.79 0) (unit 1)
     (in_bom yes) (on_board yes) (fields_autoplaced)
-    (property "Reference" "C15" (id 0) (at 177.8 95.9738 0)
+    (property "Reference" "C16" (id 0) (at 177.8 95.9738 0)
       (effects (font (size 1.27 1.27)) (justify left))
     )
@@
   (symbol (lib_id "power:GND") (at 175.26 102.87 0) (unit 1)
     (in_bom yes) (on_board yes)
-    (property "Reference" "#PWR037" (id 0) (at 175.26 109.22 0)
+    (property "Reference" "#PWR038" (id 0) (at 175.26 109.22 0)
       (effects (font (size 1.27 1.27)) hide)
     )
