File: sensors.kicad_sch (KiCad schematic)
At the start: 6 parts, among them U7 MPU-9250, U8 BMP280

Commit message: Use single connector for I/O
Parts:
- renumbered C17 to C18, C18 to C19, C19 to C20, C20 to C21
Changed lines of the file:
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@@
   (title_block
     (title "Sensors")
-    (date "2022-12-17")
+    (date "2022-12-20")
     (rev "${REVISION}")
   )
@@
   (symbol (lib_id "power:+3.3V") (at 223.52 87.63 0) (unit 1)
     (in_bom yes) (on_board yes) (fields_autoplaced)
-    (property "Reference" "#PWR044" (id 0) (at 223.52 91.44 0)
+    (property "Reference" "#PWR042" (id 0) (at 223.52 91.44 0)
       (effects (font (size 1.27 1.27)) hide)
     )
@@
   (symbol (lib_id "Device:C_Small") (at 95.25 95.25 0) (unit 1)
     (in_bom yes) (on_board yes)
-    (property "Reference" "C19" (id 0) (at 90.17 92.7162 0)
+    (property "Reference" "C20" (id 0) (at 90.17 92.7162 0)
       (effects (font (size 1.27 1.27)) (justify left))
     )
@@
   (symbol (lib_id "power:+3.3V") (at 83.82 87.63 0) (unit 1)
     (in_bom yes) (on_board yes) (fields_autoplaced)
-    (property "Reference" "#PWR043" (id 0) (at 83.82 91.44 0)
+    (property "Reference" "#PWR041" (id 0) (at 83.82 91.44 0)
       (effects (font (size 1.27 1.27)) hide)
     )
@@
   (symbol (lib_id "power:GND") (at 171.45 111.76 0) (unit 1)
     (in_bom yes) (on_board yes)
-    (property "Reference" "#PWR048" (id 0) (at 171.45 118.11 0)
+    (property "Reference" "#PWR046" (id 0) (at 171.45 118.11 0)
       (effects (font (size 1.27 1.27)) hide)
     )
@@
   (symbol (lib_id "power:GND") (at 176.53 111.76 0) (unit 1)
     (in_bom yes) (on_board yes) (fields_autoplaced)
-    (property "Reference" "#PWR049" (id 0) (at 176.53 118.11 0)
+    (property "Reference" "#PWR047" (id 0) (at 176.53 118.11 0)
       (effects (font (size 1.27 1.27)) hide)
     )
@@
   (symbol (lib_id "power:+3.3V") (at 171.45 102.87 0) (unit 1)
     (in_bom yes) (on_board yes) (fields_autoplaced)
-    (property "Reference" "#PWR046" (id 0) (at 171.45 106.68 0)
+    (property "Reference" "#PWR044" (id 0) (at 171.45 106.68 0)
       (effects (font (size 1.27 1.27)) hide)
     )
@@
   (symbol (lib_id "power:GND") (at 149.86 123.19 0) (unit 1)
     (in_bom yes) (on_board yes) (fields_autoplaced)
-    (property "Reference" "#PWR050" (id 0) (at 149.86 129.54 0)
+    (property "Reference" "#PWR048" (id 0) (at 149.86 129.54 0)
       (effects (font (size 1.27 1.27)) hide)
     )
@@
   (symbol (lib_id "power:GND") (at 223.52 110.49 0) (unit 1)
     (in_bom yes) (on_board yes) (fields_autoplaced)
-    (property "Reference" "#PWR047" (id 0) (at 223.52 116.84 0)
+    (property "Reference" "#PWR045" (id 0) (at 223.52 116.84 0)
       (effects (font (size 1.27 1.27)) hide)
     )
@@
   (symbol (lib_id "Device:C_Small") (at 176.53 107.95 0) (unit 1)
     (in_bom yes) (on_board yes) (fields_autoplaced)
-    (property "Reference" "C20" (id 0) (at 179.07 106.6862 0)
+    (property "Reference" "C21" (id 0) (at 179.07 106.6862 0)
       (effects (font (size 1.27 1.27)) (justify left))
     )
@@
   (symbol (lib_id "Device:C_Small") (at 83.82 95.25 0) (unit 1)
     (in_bom yes) (on_board yes)
-    (property "Reference" "C18" (id 0) (at 78.74 92.7162 0)
+    (property "Reference" "C19" (id 0) (at 78.74 92.7162 0)
       (effects (font (size 1.27 1.27)) (justify left))
     )
@@
   (symbol (lib_id "Device:C_Small") (at 72.39 95.25 0) (unit 1)
     (in_bom yes) (on_board yes)
-    (property "Reference" "C17" (id 0) (at 68.58 92.7162 0)
+    (property "Reference" "C18" (id 0) (at 67.31 92.7162 0)
       (effects (font (size 1.27 1.27)) (justify left))
     )
@@
   (symbol (lib_id "power:+3.3V") (at 149.86 73.66 0) (unit 1)
     (in_bom yes) (on_board yes) (fields_autoplaced)
-    (property "Reference" "#PWR042" (id 0) (at 149.86 77.47 0)
+    (property "Reference" "#PWR040" (id 0) (at 149.86 77.47 0)
       (effects (font (size 1.27 1.27)) hide)
     )
@@
   (symbol (lib_id "power:GND") (at 83.82 102.87 0) (unit 1)
     (in_bom yes) (on_board yes) (fields_autoplaced)
-    (property "Reference" "#PWR045" (id 0) (at 83.82 109.22 0)
-      (effects (font (size 1.27 1.27)) hide)
-    )
+    (property "Reference" "#PWR043" (id 0) (at 83.82 109.22 0)
+      (effects (font (size 1.27 1.27)) hide)
+    )

Commit message: Remove 5V LDO regulator
Parts:
- renumbered C18 to C16, C19 to C17, C20 to C18, C21 to C19, U7 to U6, U8 to U7
Changed lines of the file:
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@@
   (symbol (lib_id "power:+3.3V") (at 223.52 87.63 0) (unit 1)
     (in_bom yes) (on_board yes) (fields_autoplaced)
-    (property "Reference" "#PWR042" (id 0) (at 223.52 91.44 0)
+    (property "Reference" "#PWR041" (id 0) (at 223.52 91.44 0)
       (effects (font (size 1.27 1.27)) hide)
     )
@@
   (symbol (lib_id "Device:C_Small") (at 95.25 95.25 0) (unit 1)
     (in_bom yes) (on_board yes)
-    (property "Reference" "C20" (id 0) (at 90.17 92.7162 0)
+    (property "Reference" "C18" (id 0) (at 90.17 92.7162 0)
       (effects (font (size 1.27 1.27)) (justify left))
     )
@@
   (symbol (lib_id "power:+3.3V") (at 83.82 87.63 0) (unit 1)
     (in_bom yes) (on_board yes) (fields_autoplaced)
-    (property "Reference" "#PWR041" (id 0) (at 83.82 91.44 0)
+    (property "Reference" "#PWR040" (id 0) (at 83.82 91.44 0)
       (effects (font (size 1.27 1.27)) hide)
     )
@@
   (symbol (lib_id "power:GND") (at 171.45 111.76 0) (unit 1)
     (in_bom yes) (on_board yes)
-    (property "Reference" "#PWR046" (id 0) (at 171.45 118.11 0)
+    (property "Reference" "#PWR045" (id 0) (at 171.45 118.11 0)
       (effects (font (size 1.27 1.27)) hide)
     )
@@
   (symbol (lib_id "power:GND") (at 176.53 111.76 0) (unit 1)
     (in_bom yes) (on_board yes) (fields_autoplaced)
-    (property "Reference" "#PWR047" (id 0) (at 176.53 118.11 0)
+    (property "Reference" "#PWR046" (id 0) (at 176.53 118.11 0)
       (effects (font (size 1.27 1.27)) hide)
     )
@@
   (symbol (lib_id "power:+3.3V") (at 171.45 102.87 0) (unit 1)
     (in_bom yes) (on_board yes) (fields_autoplaced)
-    (property "Reference" "#PWR044" (id 0) (at 171.45 106.68 0)
+    (property "Reference" "#PWR043" (id 0) (at 171.45 106.68 0)
       (effects (font (size 1.27 1.27)) hide)
     )
@@
   (symbol (lib_id "power:GND") (at 149.86 123.19 0) (unit 1)
     (in_bom yes) (on_board yes) (fields_autoplaced)
-    (property "Reference" "#PWR048" (id 0) (at 149.86 129.54 0)
+    (property "Reference" "#PWR047" (id 0) (at 149.86 129.54 0)
       (effects (font (size 1.27 1.27)) hide)
     )
@@
   (symbol (lib_id "Sensor_Pressure:BMP280") (at 223.52 100.33 0) (unit 1)
     (in_bom yes) (on_board yes)
-    (property "Reference" "U8" (id 0) (at 215.9 91.4399 0)
+    (property "Reference" "U7" (id 0) (at 215.9 91.4399 0)
       (effects (font (size 1.27 1.27)) (justify left))
     )
@@
   (symbol (lib_id "power:GND") (at 223.52 110.49 0) (unit 1)
     (in_bom yes) (on_board yes) (fields_autoplaced)
-    (property "Reference" "#PWR045" (id 0) (at 223.52 116.84 0)
+    (property "Reference" "#PWR044" (id 0) (at 223.52 116.84 0)
       (effects (font (size 1.27 1.27)) hide)
     )
@@
   (symbol (lib_id "Device:C_Small") (at 176.53 107.95 0) (unit 1)
     (in_bom yes) (on_board yes) (fields_autoplaced)
-    (property "Reference" "C21" (id 0) (at 179.07 106.6862 0)
+    (property "Reference" "C19" (id 0) (at 179.07 106.6862 0)
       (effects (font (size 1.27 1.27)) (justify left))
     )
@@
   (symbol (lib_id "Device:C_Small") (at 83.82 95.25 0) (unit 1)
     (in_bom yes) (on_board yes)
-    (property "Reference" "C19" (id 0) (at 78.74 92.7162 0)
+    (property "Reference" "C17" (id 0) (at 78.74 92.7162 0)
       (effects (font (size 1.27 1.27)) (justify left))
     )
@@
   (symbol (lib_id "Device:C_Small") (at 72.39 95.25 0) (unit 1)
     (in_bom yes) (on_board yes)
-    (property "Reference" "C18" (id 0) (at 67.31 92.7162 0)
+    (property "Reference" "C16" (id 0) (at 67.31 92.7162 0)
       (effects (font (size 1.27 1.27)) (justify left))
     )
@@
   (symbol (lib_id "Sensor_Motion:MPU-9250") (at 149.86 99.06 0) (unit 1)
     (in_bom yes) (on_board yes)
-    (property "Reference" "U7" (id 0) (at 136.6394 80.01 0)
+    (property "Reference" "U6" (id 0) (at 136.6394 80.01 0)
       (effects (font (size 1.27 1.27)) (justify left))
     )
@@
   (symbol (lib_id "power:+3.3V") (at 149.86 73.66 0) (unit 1)
     (in_bom yes) (on_board yes) (fields_autoplaced)
-    (property "Reference" "#PWR040" (id 0) (at 149.86 77.47 0)
+    (property "Reference" "#PWR039" (id 0) (at 149.86 77.47 0)
       (effects (font (size 1.27 1.27)) hide)
     )
@@
   (symbol (lib_id "power:GND") (at 83.82 102.87 0) (unit 1)
     (in_bom yes) (on_board yes) (fields_autoplaced)
-    (property "Reference" "#PWR043" (id 0) (at 83.82 109.22 0)
-      (effects (font (size 1.27 1.27)) hide)
-    )
+    (property "Reference" "#PWR042" (id 0) (at 83.82 109.22 0)
+      (effects (font (size 1.27 1.27)) hide)
+    )

Commit message: Arrange footprints
Parts:
- renumbered C16 to C17, C17 to C18, C18 to C19, C19 to C20
Other:
- company: (none) -> Authors: H. Fedarovich, I. Kajdan
Changed lines of the file:
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@@
   (title_block
     (title "Sensors")
-    (date "2022-12-20")
+    (date "2022-12-23")
     (rev "${REVISION}")
+    (company "Authors: H. Fedarovich, I. Kajdan")
+    (comment 1 "Reviewer: A. Bondyra")
   )
   (junction (at 223.52 88.9) (diameter 0) (color 0 0 0 0)
@@
   (symbol (lib_id "power:+3.3V") (at 223.52 87.63 0) (unit 1)
     (in_bom yes) (on_board yes) (fields_autoplaced)
-    (property "Reference" "#PWR041" (id 0) (at 223.52 91.44 0)
+    (property "Reference" "#PWR042" (id 0) (at 223.52 91.44 0)
       (effects (font (size 1.27 1.27)) hide)
     )
@@
   (symbol (lib_id "Device:C_Small") (at 95.25 95.25 0) (unit 1)
     (in_bom yes) (on_board yes)
-    (property "Reference" "C18" (id 0) (at 90.17 92.7162 0)
+    (property "Reference" "C19" (id 0) (at 90.17 92.7162 0)
       (effects (font (size 1.27 1.27)) (justify left))
     )
@@
   (symbol (lib_id "power:+3.3V") (at 83.82 87.63 0) (unit 1)
     (in_bom yes) (on_board yes) (fields_autoplaced)
-    (property "Reference" "#PWR040" (id 0) (at 83.82 91.44 0)
+    (property "Reference" "#PWR041" (id 0) (at 83.82 91.44 0)
       (effects (font (size 1.27 1.27)) hide)
     )
@@
   (symbol (lib_id "power:GND") (at 171.45 111.76 0) (unit 1)
     (in_bom yes) (on_board yes)
-    (property "Reference" "#PWR045" (id 0) (at 171.45 118.11 0)
+    (property "Reference" "#PWR046" (id 0) (at 171.45 118.11 0)
       (effects (font (size 1.27 1.27)) hide)
     )
@@
   (symbol (lib_id "power:GND") (at 176.53 111.76 0) (unit 1)
     (in_bom yes) (on_board yes) (fields_autoplaced)
-    (property "Reference" "#PWR046" (id 0) (at 176.53 118.11 0)
+    (property "Reference" "#PWR047" (id 0) (at 176.53 118.11 0)
       (effects (font (size 1.27 1.27)) hide)
     )
@@
   (symbol (lib_id "power:+3.3V") (at 171.45 102.87 0) (unit 1)
     (in_bom yes) (on_board yes) (fields_autoplaced)
-    (property "Reference" "#PWR043" (id 0) (at 171.45 106.68 0)
+    (property "Reference" "#PWR044" (id 0) (at 171.45 106.68 0)
       (effects (font (size 1.27 1.27)) hide)
     )
@@
   (symbol (lib_id "power:GND") (at 149.86 123.19 0) (unit 1)
     (in_bom yes) (on_board yes) (fields_autoplaced)
-    (property "Reference" "#PWR047" (id 0) (at 149.86 129.54 0)
+    (property "Reference" "#PWR048" (id 0) (at 149.86 129.54 0)
       (effects (font (size 1.27 1.27)) hide)
     )
@@
   (symbol (lib_id "power:GND") (at 223.52 110.49 0) (unit 1)
     (in_bom yes) (on_board yes) (fields_autoplaced)
-    (property "Reference" "#PWR044" (id 0) (at 223.52 116.84 0)
+    (property "Reference" "#PWR045" (id 0) (at 223.52 116.84 0)
       (effects (font (size 1.27 1.27)) hide)
     )
@@
   (symbol (lib_id "Device:C_Small") (at 176.53 107.95 0) (unit 1)
     (in_bom yes) (on_board yes) (fields_autoplaced)
-    (property "Reference" "C19" (id 0) (at 179.07 106.6862 0)
+    (property "Reference" "C20" (id 0) (at 179.07 106.6862 0)
       (effects (font (size 1.27 1.27)) (justify left))
     )
@@
   (symbol (lib_id "Device:C_Small") (at 83.82 95.25 0) (unit 1)
     (in_bom yes) (on_board yes)
-    (property "Reference" "C17" (id 0) (at 78.74 92.7162 0)
+    (property "Reference" "C18" (id 0) (at 78.74 92.7162 0)
       (effects (font (size 1.27 1.27)) (justify left))
     )
@@
   (symbol (lib_id "Device:C_Small") (at 72.39 95.25 0) (unit 1)
     (in_bom yes) (on_board yes)
-    (property "Reference" "C16" (id 0) (at 67.31 92.7162 0)
+    (property "Reference" "C17" (id 0) (at 67.31 92.7162 0)
       (effects (font (size 1.27 1.27)) (justify left))
     )
@@
   (symbol (lib_id "power:+3.3V") (at 149.86 73.66 0) (unit 1)
     (in_bom yes) (on_board yes) (fields_autoplaced)
-    (property "Reference" "#PWR039" (id 0) (at 149.86 77.47 0)
+    (property "Reference" "#PWR040" (id 0) (at 149.86 77.47 0)
       (effects (font (size 1.27 1.27)) hide)
     )
@@
   (symbol (lib_id "power:GND") (at 83.82 102.87 0) (unit 1)
     (in_bom yes) (on_board yes) (fields_autoplaced)
-    (property "Reference" "#PWR042" (id 0) (at 83.82 109.22 0)
-      (effects (font (size 1.27 1.27)) hide)
-    )
+    (property "Reference" "#PWR043" (id 0) (at 83.82 109.22 0)
+      (effects (font (size 1.27 1.27)) hide)
+    )
